File: hardware/open_gamma_low_noise.kicad_sch (KiCad schematic)
At the start: 62 parts, among them J1 1909763-1, J2 1909763-1, Q1 2N7002,215, U1 TLV3201AIDBVR, U2 LM4040AIM3-3.0+T, U3 Pico, U4 OPA357AIDBVTG4, U5 MAX5026EUT+T, U6 LM4040AIM3-3.0+T, U7 OPA357AIDBVTG4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

Commit message: Update open_gamma_low_noise.kicad_sch
Other:
- company: (none) -> Gigstorm
- title: (none) -> Open Gamma Low Noise
Changed lines of the file:
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@@
 (kicad_sch (version 20230121) (generator eeschema)
   (paper "A4")
+  (title_block
+    (title "Open Gamma Low Noise")
+    (date "2023-07-25")
+    (rev "3a")
+    (company "Gigstorm")
+  )
   (junction (at 247.65 53.34) (diameter 0) (color 0 0 0 0)
   )

Commit message: Updated 3D models
Parts:
- I2C1, SPI1: footprint Connector_PinSocket_2.54mm:PinSocket_1x04_P2.54mm_Vertical -> Connector_PinHeader_2.54mm:PinHeader_1x04_P2.54mm_Vertical
- J3: footprint Connector_PinSocket_2.54mm:PinSocket_1x03_P2.54mm_Vertical -> Connector_PinHeader_2.54mm:PinHeader_1x03_P2.54mm_Vertical
- R2, R8: footprint 3296W-1-103:3296W1103 -> Trimmer_Res:POT_3296W
- UART1: footprint Connector_PinSocket_2.54mm:PinSocket_1x02_P2.54mm_Vertical -> Connector_PinHeader_2.54mm:PinHeader_1x02_P2.54mm_Vertical
Changed lines of the file:
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@@
       (effects (font (size 1.27 1.27)) (justify right))
     )
-    (property "Footprint" "3296W-1-103:3296W1103" (at 139.7 27.94 0)
+    (property "Footprint" "Trimmer_Res:POT_3296W" (at 139.7 27.94 0)
       (effects (font (size 1.27 1.27)) hide)
     )
@@
       (effects (font (size 1.27 1.27)) (justify left) hide)
     )
-    (property "Footprint" "Connector_PinSocket_2.54mm:PinSocket_1x02_P2.54mm_Vertical" (at 97.79 120.65 0)
+    (property "Footprint" "Connector_PinHeader_2.54mm:PinHeader_1x02_P2.54mm_Vertical" (at 97.79 120.65 0)
       (effects (font (size 1.27 1.27)) hide)
     )
@@
       (effects (font (size 1.27 1.27)) hide)
     )
-    (property "Footprint" "Connector_PinSocket_2.54mm:PinSocket_1x04_P2.54mm_Vertical" (at 99.06 100.33 0)
+    (property "Footprint" "Connector_PinHeader_2.54mm:PinHeader_1x04_P2.54mm_Vertical" (at 99.06 100.33 0)
       (effects (font (size 1.27 1.27)) hide)
     )
@@
       (effects (font (size 1.27 1.27)))
     )
-    (property "Footprint" "Connector_PinSocket_2.54mm:PinSocket_1x04_P2.54mm_Vertical" (at 73.66 104.14 0)
+    (property "Footprint" "Connector_PinHeader_2.54mm:PinHeader_1x04_P2.54mm_Vertical" (at 73.66 104.14 0)
       (effects (font (size 1.27 1.27)) hide)
     )
@@
       (effects (font (size 1.27 1.27)))
     )
-    (property "Footprint" "Connector_PinSocket_2.54mm:PinSocket_1x03_P2.54mm_Vertical" (at 214.63 90.17 0)
+    (property "Footprint" "Connector_PinHeader_2.54mm:PinHeader_1x03_P2.54mm_Vertical" (at 214.63 90.17 0)
       (effects (font (size 1.27 1.27)) hide)
     )
@@
       (effects (font (size 1.27 1.27)) (justify right))
     )
-    (property "Footprint" "3296W-1-103:3296W1103" (at 71.12 157.48 0)
-      (effects (font (size 1.27 1.27)) hide)
-    )
+    (property "Footprint" "Trimmer_Res:POT_3296W" (at 71.12 157.48 0)
+      (effects (font (size 1.27 1.27)) hide)
+    )
